File: OpenSprinkler Controller/hardware/v2.0/smt/os20.newenc.sch (EAGLE design)
At the start: 44 parts, among them IC1 LM2596S-5.0, IC2 LM1117-33, IC3 DS1307, IC6 ENC28J60, IC7 ATTINY45SO8S2, J0 24VAC IN, J2 EG1206, U1 ATMEGA328P, U2 LCD-16X2SILK, X1 25MHz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

Commit message: pakeistas lcd i nokia
Parts:
- removed U2: LCD-16X2SILK, SparkFun-Displays:LCD-16X2SILK
- added S1, S2, S3, S4, S5: (no value), SparkFun-Electromechanical:TAC_SWITCHPTH
- added U$2: CELLPHONE_NOKIA_5100, DIY-Cellphone:CELLPHONE_NOKIA_5100
Connections:
- removed net D18: U2.DB4
- removed net D20: U2.E
- removed net D21: U2.R/W
- removed net D22: U2.RS
- removed net D23: U2.VO
- net D12: no longer U2.VSS
- net GND: no longer U2.A, U2.DB5, U2.DB6, U2.DB7, U2.K
- net VIN: no longer U2.VDD
Changed lines of the file:
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@@
 <part name="IC1" library="national-semiconductor" deviceset="LM2596" device="S" value="LM2596S-5.0"/>
 <part name="U1" library="SparkFun-DigitalIC" deviceset="ATMEGA328_SMT" device="" value="ATMEGA328P"/>
-<part name="U2" library="SparkFun-Displays" deviceset="LCD-16X2" device="SILK" value="LCD-16X2SILK"/>
+<part name="U$2" library="DIY-Cellphone" deviceset="CELLPHONE_NOKIA_5100" device=""/>
+<part name="S1" library="SparkFun-Electromechanical" deviceset="TAC_SWITCH" device="PTH"/>
+<part name="S2" library="SparkFun-Electromechanical" deviceset="TAC_SWITCH" device="PTH"/>
+<part name="S3" library="SparkFun-Electromechanical" deviceset="TAC_SWITCH" device="PTH"/>
+<part name="S4" library="SparkFun-Electromechanical" deviceset="TAC_SWITCH" device="PTH"/>
+<part name="S5" library="SparkFun-Electromechanical" deviceset="TAC_SWITCH" device="PTH"/>
 </parts>
 <sheets>
@@
 <instance part="IC1" gate="G$1" x="26.67" y="152.4"/>
 <instance part="U1" gate="G$1" x="187.96" y="86.36"/>
-<instance part="U2" gate="G$1" x="119.38" y="157.48"/>
+<instance part="U$2" gate="G$1" x="-71.12" y="144.78"/>
+<instance part="S1" gate="S" x="-20.32" y="223.52"/>
+<instance part="S2" gate="S" x="-7.62" y="223.52"/>
+<instance part="S3" gate="S" x="5.08" y="223.52"/>
+<instance part="S4" gate="S" x="17.78" y="223.52"/>
+<instance part="S5" gate="S" x="33.02" y="223.52"/>
 </instances>
 <busses>
@@
 <pinref part="D3" gate="G$1" pin="A"/>
 <junction x="40.64" y="139.7"/>
-<pinref part="U2" gate="G$1" pin="A"/>
-<junction x="109.22" y="142.24"/>
-<pinref part="U2" gate="G$1" pin="DB5"/>
-<junction x="109.22" y="149.86"/>
-<pinref part="U2" gate="G$1" pin="DB6"/>
-<junction x="109.22" y="147.32"/>
-<pinref part="U2" gate="G$1" pin="DB7"/>
-<junction x="109.22" y="144.78"/>
-<pinref part="U2" gate="G$1" pin="K"/>
 </segment>
 <segment>
@@
 <pinref part="GND16" gate="1" pin="GND"/>
 </segment>
+<segment>
+<wire x1="-66.04" y1="172.72" x2="-71.12" y2="172.72" width="0.1524" layer="91"/>
+<label x="-71.12" y="172.72" size="1.778" layer="95"/>
+</segment>
 </net>
 <net name="RESET" class="0">
@@
 <label x="170.18" y="30.48" size="1.778" layer="95"/>
 <pinref part="ISP" gate="A" pin="3"/>
+</segment>
+<segment>
+<wire x1="-66.04" y1="195.58" x2="-73.66" y2="195.58" width="0.1524" layer="91"/>
+<label x="-73.66" y="195.58" size="1.778" layer="95"/>
 </segment>
 </net>
@@
 <junction x="73.66" y="154.94"/>
 <pinref part="F1" gate="G$1" pin="2"/>
-<pinref part="U2" gate="G$1" pin="VDD"/>
-<junction x="109.22" y="175.26"/>
 </segment>
 <segment>
@@
 <wire x1="110.49" y1="172.72" x2="109.22" y2="172.72" width="0.1524" layer="91"/>
 <label x="102.87" y="172.72" size="1.778" layer="95"/>
-<pinref part="U2" gate="G$1" pin="VO"/>
 <wire x1="109.22" y1="172.72" x2="102.87" y2="172.72" width="0.1524" layer="91"/>
-<junction x="109.22" y="172.72"/>
 </segment>
 </net>
@@
 <wire x1="110.49" y1="170.18" x2="109.22" y2="170.18" width="0.1524" layer="91"/>
 <label x="102.87" y="170.18" size="1.778" layer="95"/>
-<pinref part="U2" gate="G$1" pin="RS"/>
 <wire x1="109.22" y1="170.18" x2="102.87" y2="170.18" width="0.1524" layer="91"/>
-<junction x="109.22" y="170.18"/>
 </segment>
 </net>
@@
 <wire x1="110.49" y1="167.64" x2="109.22" y2="167.64" width="0.1524" layer="91"/>
 <label x="102.87" y="167.64" size="1.778" layer="95"/>
-<pinref part="U2" gate="G$1" pin="R/W"/>
 <wire x1="109.22" y1="167.64" x2="102.87" y2="167.64" width="0.1524" layer="91"/>
-<junction x="109.22" y="167.64"/>
 </segment>
 </net>
@@
 <wire x1="110.49" y1="165.1" x2="109.22" y2="165.1" width="0.1524" layer="91"/>
 <label x="102.87" y="165.1" size="1.778" layer="95"/>
-<pinref part="U2" gate="G$1" pin="E"/>
 <wire x1="109.22" y1="165.1" x2="102.87" y2="165.1" width="0.1524" layer="91"/>
-<junction x="109.22" y="165.1"/>
 </segment>
 </net>
@@
 <wire x1="110.49" y1="152.4" x2="109.22" y2="152.4" width="0.1524" layer="91"/>
 <label x="102.87" y="152.4" size="1.778" layer="95"/>
-<pinref part="U2" gate="G$1" pin="DB4"/>
 <wire x1="109.22" y1="152.4" x2="102.87" y2="152.4" width="0.1524" layer="91"/>
-<junction x="109.22" y="152.4"/>
 </segment>
 </net>
@@
 <wire x1="102.87" y1="177.8" x2="109.22" y2="177.8" width="0.1524" layer="91"/>
 <label x="102.87" y="177.8" size="1.778" layer="95"/>
-<pinref part="U2" gate="G$1" pin="VSS"/>
 <wire x1="109.22" y1="177.8" x2="110.49" y2="177.8" width="0.1524" layer="91"/>
-<junction x="109.22" y="177.8"/>
 </segment>
 <segment>
@@
 </segment>
 </net>
+<net name="CS" class="0">
+<segment>
+<wire x1="-66.04" y1="190.5" x2="-73.66" y2="190.5" width="0.1524" layer="91"/>
+<label x="-73.66" y="190.5" size="1.778" layer="95"/>
+</segment>
+</net>
+<net name="DIO" class="0">
+<segment>
+<wire x1="-66.04" y1="193.04" x2="-73.66" y2="193.04" width="0.1524" layer="91"/>
+<label x="-73.66" y="193.04" size="1.778" layer="95"/>
+</segment>
+</net>
