File: OpenSprinkler Controller/hardware/v2.0/smt/os20.newenc.sch (EAGLE design)
At the start: 49 parts, among them IC1 LM2596S-5.0, IC2 LM1117-33, IC3 DS1307, IC6 ENC28J60, IC7 ATTINY45SO8S2, J0 24VAC IN, J2 EG1206, U1 ATMEGA328P, X1 25MHz, X2 32.768kHz

Commit message: Pakeista Nokia LCD biblioteka
Connections:
- new net N$23: U$2.CE
- new net N$24: U$2.DC
- new net N$25: U$2.DIN
- new net V$: U$2.RST
- net GND: now also U$2.GND
- net VCC: now also U$2.VCC
Other:
- moved on the sheet: U$2
Changed lines of the file:
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@@
 <setting verticaltext="up"/>
 </settings>
-<grid distance="0.254" unitdist="mm" unit="mm" style="lines" multiple="1" display="no" altdistance="0.01" altunitdist="inch" altunit="mm"/>
+<grid distance="1.27" unitdist="mm" unit="mm" style="lines" multiple="1" display="yes" altdistance="0.01" altunitdist="inch" altunit="mm"/>
 <layers>
 <layer number="1" name="Top" color="4" fill="1" visible="no" active="no"/>
@@
 <instance part="IC1" gate="G$1" x="26.67" y="152.4"/>
 <instance part="U1" gate="G$1" x="187.96" y="86.36"/>
-<instance part="U$2" gate="G$1" x="89.916" y="201.168" rot="R270"/>
+<instance part="U$2" gate="G$1" x="92.71" y="198.12" rot="R270"/>
 <instance part="S1" gate="S" x="-20.32" y="223.52"/>
 <instance part="S2" gate="S" x="-7.62" y="223.52"/>
@@
 <junction x="121.92" y="67.31"/>
 </segment>
+<segment>
+<pinref part="U$2" gate="G$1" pin="GND"/>
+<wire x1="105.41" y1="190.5" x2="111.76" y2="190.5" width="0.1524" layer="91"/>
+</segment>
 </net>
 <net name="RESET" class="0">
@@
 <junction x="-8.89" y="86.36"/>
 </segment>
+<segment>
+<pinref part="U$2" gate="G$1" pin="VCC"/>
+<wire x1="105.41" y1="195.58" x2="111.76" y2="195.58" width="0.1524" layer="91"/>
+</segment>
 </net>
 <net name="TCT" class="0">
@@
 </segment>
 </net>
+<net name="N$23" class="0">
+<segment>
+<pinref part="U$2" gate="G$1" pin="CE"/>
+<wire x1="105.41" y1="205.74" x2="109.22" y2="205.74" width="0.1524" layer="91"/>
+</segment>
+</net>
+<net name="N$24" class="0">
+<segment>
+<pinref part="U$2" gate="G$1" pin="DC"/>
+<wire x1="105.41" y1="203.2" x2="109.22" y2="203.2" width="0.1524" layer="91"/>
+</segment>
+</net>
+<net name="N$25" class="0">
+<segment>
+<pinref part="U$2" gate="G$1" pin="DIN"/>
+<wire x1="105.41" y1="200.66" x2="109.22" y2="200.66" width="0.1524" layer="91"/>
+</segment>
+</net>
+<net name="V$" class="0">
+<segment>
+<wire x1="105.41" y1="208.28" x2="109.22" y2="208.28" width="0.1524" layer="91"/>
+<pinref part="U$2" gate="G$1" pin="RST"/>
+<label x="106.68" y="208.28" size="1.778" layer="95"/>
+</segment>
+</net>

Commit message: pirmyn...
Parts:
- added R1, R2, R3, R4, R5, R6: 10k, rcl:R-EU_R0805
- renumbered RD+ to R8, RD- to R7
Connections:
- removed net N$17: U1.PD3(INT1)
- removed net N$18: U1.PD4(XCK/T0)
- removed net N$19: U1.PD5(T1)
- removed net N$20: U1.PD6(AIN0)
- removed net N$21: U1.PD7(AIN1)
- new net D3: R2.2, U1.PD3(INT1)
- new net D4: R3.2, U1.PD4(XCK/T0)
- new net D5: R4.2, U1.PD5(T1)
- new net D6: R6.2, U1.PD6(AIN0)
- new net D7: R5.2, U1.PD7(AIN1)
- new net N$22: R2.1, U$2.CLK
- new net N$26: R1.1, U$2.BL
- new net N$51: R1.2
- net N$23: now also R5.1
- net N$24: now also R4.1
- net N$25: now also R3.1
- net V$: now also R6.1
