File: OpenSprinkler Controller/hardware/v2.0/smt/os20.newenc.brd (EAGLE design)
At the start: 100 x 50 mm, 44 parts, among them IC1 LM2596S-5.0, IC2 LM1117-33, IC3 DS1307, IC6 ENC28J60, IC7 ATTINY45SO8S2, J0 24VAC IN, J2 EG1206, U1 ATMEGA328P, U2 LCD-16X2SILK, X1 25MHz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

Commit message: pakeistas lcd i nokia
Parts:
- removed U2: LCD-16X2SILK, SparkFun-Displays:LCD-16X2
- added S1, S2, S3, S4, S5: (no value), SparkFun-Electromechanical:TACTILE-PTH
- added U$2: CELLPHONE_NOKIA_5100, DIY-Cellphone:CELLPHONE_NOKIA_5100_SPARKFUN
- moved RJ45 74.1 mm to (55.2, 43.2), turned to 90 degrees
- moved CAP 69.4 mm to (125.5, 1.06)
- moved U1 68.9 mm to (130.8, 16.5)
- moved IC6 52.2 mm to (122.1, 33.2)
Connections:
- removed net D18: U2.11
- removed net D20: U2.6
- removed net D21: U2.5
- removed net D22: U2.4
- removed net D23: U2.3
- net D12: no longer U2.1
- net GND: no longer U2.12, U2.13, U2.14, U2.15, U2.16
- net VIN: no longer U2.2
Other:
- board text removed: "GND A3 VIN"
- board text removed: "GND VIN A3"

Commit message: smulkmenos..
Parts:
- USB: value USBPTH -> (none); device SparkFunNew:USB-B-PTH -> adafruit:USB-MINIB-THM-MOLEX
- moved USB 80.7 mm to (52.5, -1.93)
- moved BAT1 30.2 mm to (13.6, 83.4)
- moved IC2 11.7 mm to (-29.4, 51.5)
- moved L1 11.4 mm to (-26.9, -13.8)
- moved D1 10.2 mm to (-40.5, 21.2)
- moved D3 7.41 mm to (-47.0, 11.8)
- moved IC1 6.35 mm to (-14.5, 18.7)
Connections:
- net GND: now also USB.ID

Commit message: Pakeista Nokia LCD biblioteka
Connections:
- new net N$23: U$2.P$2
- new net N$24: U$2.P$3
- new net N$25: U$2.P$4
- new net V$: U$2.P$1
- net GND: now also U$2.P$8
- net VCC: now also U$2.P$6
Changed lines of the file:
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@@
 <contactref element="D3" pad="A"/>
 <contactref element="USB" pad="ID"/>
+<contactref element="U$2" pad="P$8"/>
 <wire x1="121.745" y1="36.846" x2="122.395" y2="36.846" width="0" layer="19" extent="1-1"/>
 <wire x1="124.345" y1="36.846" x2="122.395" y2="36.846" width="0" layer="19" extent="1-1"/>
@@
 <wire x1="68.7" y1="-5.29" x2="80.77" y2="-1.91" width="0" layer="19" extent="1-1"/>
 <wire x1="68.58" y1="-15.75" x2="68.7" y2="-5.29" width="0" layer="19" extent="1-1"/>
-<wire x1="40.365" y1="-27.1982" x2="68.58" y2="-15.75" width="0" layer="19" extent="1-1"/>
-<wire x1="6.95" y1="-6.15" x2="40.365" y2="-27.1982" width="0" layer="19" extent="1-1"/>
-<wire x1="4.7" y1="3.522" x2="6.95" y2="-6.15" width="0" layer="19" extent="1-1"/>
-<wire x1="-11.1244" y1="12.9208" x2="4.7" y2="3.522" width="0" layer="19" extent="1-1"/>
-<wire x1="-14.528" y1="12.9208" x2="-11.1244" y2="12.9208" width="0" layer="19" extent="1-1"/>
-<wire x1="-27.18" y1="4.73" x2="-14.528" y2="12.9208" width="0" layer="19" extent="1-1"/>
-<wire x1="-34.96" y1="8.7" x2="-27.18" y2="4.73" width="0" layer="19" extent="1-1"/>
-<wire x1="-45.015" y1="11.76" x2="-34.96" y2="8.7" width="0" layer="19" extent="1-1"/>
-<wire x1="53.25" y1="6.49" x2="-11.1244" y2="12.9208" width="0" layer="19" extent="1-1"/>
+<wire x1="53.25" y1="6.49" x2="68.7" y2="-5.29" width="0" layer="19" extent="1-1"/>
 <wire x1="54.05" y1="7.79" x2="53.25" y2="6.49" width="0" layer="19" extent="1-1"/>
-<wire x1="-27.1086" y1="54.5688" x2="54.05" y2="7.79" width="0" layer="19" extent="1-1"/>
-<wire x1="14.397" y1="57.4346" x2="-27.1086" y2="54.5688" width="0" layer="19" extent="1-1"/>
-<wire x1="13.188" y1="66.254" x2="14.397" y2="57.4346" width="0" layer="19" extent="1-1"/>
-<wire x1="25.53" y1="83.44" x2="14.397" y2="57.4346" width="0" layer="19" extent="1-1"/>
-<wire x1="38.7" y1="43" x2="25.53" y2="83.44" width="0" layer="19" extent="1-1"/>
-<wire x1="47.239" y1="40.279" x2="38.7" y2="43" width="0" layer="19" extent="1-1"/>
-<wire x1="50.795" y1="34.31" x2="47.239" y2="40.279" width="0" layer="19" extent="1-1"/>
+<wire x1="50.795" y1="34.31" x2="54.05" y2="7.79" width="0" layer="19" extent="1-1"/>
+<wire x1="47.239" y1="40.279" x2="50.795" y2="34.31" width="0" layer="19" extent="1-1"/>
 <wire x1="51.176" y1="48.153" x2="47.239" y2="40.279" width="0" layer="19" extent="1-1"/>
 <wire x1="59.304" y1="48.153" x2="51.176" y2="48.153" width="0" layer="19" extent="1-1"/>
@@
 <wire x1="55.05" y1="62" x2="52.324" y2="56.68" width="0" layer="19" extent="1-1"/>
 <wire x1="63.241" y1="40.279" x2="59.304" y2="48.153" width="0" layer="19" extent="1-1"/>
+<wire x1="38.7" y1="43" x2="47.239" y2="40.279" width="0" layer="19" extent="1-1"/>
+<wire x1="31.75" y1="46.67" x2="38.7" y2="43" width="0" layer="19" extent="1-1"/>
+<wire x1="14.397" y1="57.4346" x2="31.75" y2="46.67" width="0" layer="19" extent="1-1"/>
+<wire x1="13.188" y1="66.254" x2="14.397" y2="57.4346" width="0" layer="19" extent="1-1"/>
+<wire x1="25.53" y1="83.44" x2="13.188" y2="66.254" width="0" layer="19" extent="1-1"/>
+<wire x1="40.365" y1="-27.1982" x2="68.58" y2="-15.75" width="0" layer="19" extent="1-1"/>
+<wire x1="6.95" y1="-6.15" x2="40.365" y2="-27.1982" width="0" layer="19" extent="1-1"/>
+<wire x1="4.7" y1="3.522" x2="6.95" y2="-6.15" width="0" layer="19" extent="1-1"/>
+<wire x1="-11.1244" y1="12.9208" x2="4.7" y2="3.522" width="0" layer="19" extent="1-1"/>
+<wire x1="-14.528" y1="12.9208" x2="-11.1244" y2="12.9208" width="0" layer="19" extent="1-1"/>
+<wire x1="-27.18" y1="4.73" x2="-14.528" y2="12.9208" width="0" layer="19" extent="1-1"/>
+<wire x1="-34.96" y1="8.7" x2="-27.18" y2="4.73" width="0" layer="19" extent="1-1"/>
+<wire x1="-45.015" y1="11.76" x2="-34.96" y2="8.7" width="0" layer="19" extent="1-1"/>
+<wire x1="-27.1086" y1="54.5688" x2="14.397" y2="57.4346" width="0" layer="19" extent="1-1"/>
 </signal>
 <signal name="RESET">
@@
 <contactref element="C6" pad="1"/>
 <contactref element="RN4" pad="6"/>
-<wire x1="126.295" y1="36.846" x2="80.05" y2="-10.8" width="0" layer="19" extent="1-1"/>
+<contactref element="U$2" pad="P$6"/>
 <wire x1="123.695" y1="36.846" x2="126.295" y2="36.846" width="0" layer="19" extent="1-1"/>
 <wire x1="123.045" y1="36.846" x2="123.695" y2="36.846" width="0" layer="19" extent="1-1"/>
 <wire x1="119.795" y1="36.846" x2="123.045" y2="36.846" width="0" layer="19" extent="1-1"/>
 <wire x1="117.845" y1="36.846" x2="119.795" y2="36.846" width="0" layer="19" extent="1-1"/>
-<wire x1="57.86" y1="52.89" x2="117.845" y2="36.846" width="0" layer="19" extent="1-1"/>
-<wire x1="56.95" y1="62" x2="57.86" y2="52.89" width="0" layer="19" extent="1-1"/>
-<wire x1="44.4" y1="59.75" x2="56.95" y2="62" width="0" layer="19" extent="1-1"/>
-<wire x1="-29.42" y1="48.371" x2="44.4" y2="59.75" width="0" layer="19" extent="1-1"/>
-<wire x1="6.95" y1="-1.35" x2="-29.42" y2="48.371" width="0" layer="19" extent="1-1"/>
+<wire x1="80.05" y1="-10.8" x2="117.845" y2="36.846" width="0" layer="19" extent="1-1"/>
+<wire x1="36.555" y1="-19.5672" x2="80.05" y2="-10.8" width="0" layer="19" extent="1-1"/>
+<wire x1="6.95" y1="-1.35" x2="36.555" y2="-19.5672" width="0" layer="19" extent="1-1"/>
 <wire x1="-1.15" y1="-12.8" x2="6.95" y2="-1.35" width="0" layer="19" extent="1-1"/>
-<wire x1="36.555" y1="-19.5672" x2="6.95" y2="-1.35" width="0" layer="19" extent="1-1"/>
+<wire x1="26.67" y1="46.67" x2="6.95" y2="-1.35" width="0" layer="19" extent="1-1"/>
+<wire x1="44.4" y1="59.75" x2="26.67" y2="46.67" width="0" layer="19" extent="1-1"/>
+<wire x1="56.95" y1="62" x2="44.4" y2="59.75" width="0" layer="19" extent="1-1"/>
+<wire x1="57.86" y1="52.89" x2="56.95" y2="62" width="0" layer="19" extent="1-1"/>
+<wire x1="-29.42" y1="48.371" x2="26.67" y2="46.67" width="0" layer="19" extent="1-1"/>
 </signal>
 <signal name="TCT">
@@
 <wire x1="135.1026" y1="18.51" x2="121.745" y2="29.534" width="0" layer="19" extent="1-1"/>
 </signal>
+<signal name="N$23">
+<contactref element="U$2" pad="P$2"/>
+</signal>
+<signal name="N$24">
+<contactref element="U$2" pad="P$3"/>
+</signal>
+<signal name="N$25">
+<contactref element="U$2" pad="P$4"/>
+</signal>
+<signal name="V$">
+<contactref element="U$2" pad="P$1"/>
+</signal>
 </signals>

Commit message: pirmyn...
Parts:
- removed RD+, RD-: 47, rcl:R0805
- added R1, R2, R3, R4, R5, R6: 10k, rcl:R0805
- added R7, R8: 47, rcl:R0805
- moved CAP 119.2 mm to (9.12, 26.9), turned to 180 degrees
- moved IC6 111.9 mm to (11.3, 17.6), turned to 180 degrees
- moved U1 104.8 mm to (26.7, 27.9), turned to 270 degrees
- moved C8 84.1 mm to (8.98, 30.7), turned to 0 degrees
- moved REA 71.8 mm to (20.3, 13.5)
- moved C7 60.7 mm to (22.8, 18.4)
- moved C4 58.5 mm to (107.1, 19.9)
- moved USB 56.0 mm to (69.5, 51.5), turned to 180 degrees
- moved IC7 54.0 mm to (62.6, 24.8)
- moved CX1 49.0 mm to (108.4, 25.4)
- moved C5 45.6 mm to (108.5, 41.8)
- moved CX2 38.7 mm to (111.1, 36.9)
- moved RN3 34.2 mm to (49.0, 19.5)
- moved ISP 26.9 mm to (49.8, 27.5)
- moved IC3 24.5 mm to (3.60, 37.6)
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Connections:
- removed net N$17: U1.1
- removed net N$18: U1.2
- removed net N$19: U1.9
- removed net N$20: U1.10
- removed net N$21: U1.11
- new net D3: R2.2, U1.1
- new net D4: R3.2, U1.2
- new net D5: R4.2, U1.9
- new net D6: R6.2, U1.10
- new net D7: R5.2, U1.11
- new net N$22: R2.1, U$2.P$5
- new net N$26: R1.1, U$2.P$7
- new net N$51: R1.2
- net D+: now also R8.1; no longer RD+.1
- net D-: now also R7.1; no longer RD-.1
- net N$23: now also R5.1
- net N$24: now also R4.1
- net N$25: now also R3.1
- net N$38: now also R8.2; no longer RD+.2
- net N$45: now also R7.2; no longer RD-.2
- net V$: now also R6.1
